File: MIDIpod.brd (EAGLE design)
At the start: 45 x 85 mm, 59 parts, among them IC1 TPA6132A2, J1 SJ-3524-SMT-TR, J4 68610814122, Q1 MMUN2133LT1G, Q2 9.6MHz, U1 TPS61090RSAR, U2 MCP73831T-2ACI/OT

Commit message: updated, sent to oshpark
Parts:
- removed B1: 1.8-5V, microbuilder:JSTPH2
- removed CA11, CA12: 2.2uf, rcl:C0603
- removed IC1: TPA6132A2, texas:QFN16
- removed JP1: (no value), pinhead:1X03
- removed L1: VLC5045-6.8uH, microbuilder:INDUCTOR_5X5MM_TDK_VLC5045
- removed LBO: RED, microbuilder:CHIPLED_0805_NOOUTLINE
- removed PWR: BLUE, microbuilder:CHIPLED_0805_NOOUTLINE
- removed Q1: MMUN2133LT1G, transistor:SC59-BEC
- removed Q2: 9.6MHz, crystal:TC26H
- removed SD1: MF-MICROSD, MF_Connectors:MF-MICROSD
- removed U$10, U$12, U$35, U$36: 1U_PAD, SiliconeSwitches:SILICONE_SWITCH
- removed U$13: ATMEGA32U4-AU, adafruit:TQFP44
- added BUTTON1, BUTTON2, BUTTON3, BUTTON4, BUTTON5: 1U_PAD, SiliconeSwitches:SILICONE_SWITCH
- added C10, C9: 2.2pF, rcl:C0603
- added C11, C12: 2.2uf, rcl:C0603
- added C13, C14: 1uF, SparkFun-Capacitors:0402
- added CD2, CD3: 22pf, rcl:C0603
- added D2: MBR120, diode:SMB
- added ISP1: AVRISP-6, adafruit:AVRISP
- added J2: (no value), SparkFun-Connectors:1X02
- added POWER_SW: ALPSSLIDESW, TindieBadge:SWITCH-SSSS810701
- added R10: 10k, rcl:R0603
- added R21: 1k, rcl:R0603
- added R22: 220, rcl:R0603
- added R9: 100k, microbuilder:0805-NO
- added U3: SPX3819M5_3_3, SparkFun-IC-Power:SOT23-5
- added U_CTRL: ATMEGA32U4-AU, adafruit:TQFP44
- added U_SD: MICROSD, adafruit:MICROSD
- added Y1: 16MHz, SparkFun-Clocks:CRYSTAL-SMD-3.2X1.5MM
- added Y2: 9.6MHz, SparkFun-Clocks:CRYSTAL-SMD-3.2X1.5MM
- C3: value 10uF -> 10µF
- C5: value 2.2uF -> 10µF
- C7: value 0.1uF -> 1uF
- C8: value 100uF/6V -> 2.2uF; device microbuilder:EIA3528-21/B-R -> SparkFun-Capacitors:0805
- R15: value 1K -> 10k; device microbuilder:0805-NO -> rcl:R0603
- R16: value 1.87Mohm -> 10k; device microbuilder:0805-NO -> rcl:R0603
- R17: value 200K -> 10k; device microbuilder:0805-NO -> rcl:R0603
- R18: value 340K -> 220; device microbuilder:0805-NO -> rcl:R0603
- R19: value 1.87Mohm -> 22; device microbuilder:0805-NO -> rcl:R0603
- R2: value 0 -> 220
- R20: value 1K -> 22; device microbuilder:0805-NO -> rcl:R0603
- U1: value TPS61090RSAR -> TPA6111A2DR; device microbuilder:PVQFN-16 -> SparkFun-IC-Amplifiers:SO08
- moved R6 95.7 mm to (25.7, 44.4), flipped to the bottom, turned to 90 degrees
- moved R5 85.5 mm to (24.0, 38.2), flipped to the bottom
- moved CD1 79.4 mm to (16.7, 31.6), flipped to the bottom
- moved CD5 74.3 mm to (5.93, 35.8), flipped to the bottom
- moved R3 63.9 mm to (23.6, 44.3), flipped to the bottom, turned to 270 degrees
- moved U$1 55.3 mm to (17.9, 37.5)
- moved R8 55.2 mm to (23.9, 39.8)
- moved R12 55.1 mm to (24.0, 33.5)
- moved C4 54.7 mm to (24.0, 35.1)
- moved D1 54.3 mm to (24.2, 31.6)
- moved R7 53.3 mm to (19.7, 44.4), turned to 270 degrees
- moved R1 53.1 mm to (21.6, 44.3), turned to 90 degrees
- moved CA6 53.1 mm to (17.8, 44.3)
- moved CA2 53.0 mm to (15.7, 44.4)
- moved C2 52.6 mm to (9.34, 36.9)
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Connections:
- removed net 3.3V: SD1.PIN4
- removed net 5.0V: C5.1, C8.+, PWR.A, R16.2, U1.1, U1.15, U1.16
- removed net AGND: CA2.2, CA6.2, R2.2, R3.1, R7.1, U$1.P42, U$1.P43, U$1.P44
- removed net LBO: Q1.B, U1.12
- removed net LCD_K: J3.2
- removed net PGND: IC1.10
- removed net PIN4: JP1.1
- removed net SGND: IC1.15
- removed net TXD: JP1.3
- removed net VDD: IC1.14
- removed net VDD1: C6.1, LED3.A, U$43.A4B9, U$43.B4A9, U2.4
- new net 7: U_CTRL.1, U_SD.CD1
- new net LCD_CAP1N: C8.2, J4.7
- new net LCD_CAP1P: C8.1, J4.6
- new net LCD_SCL: J4.2, U_CTRL.18
- new net LCD_SDA: J4.3, U_CTRL.19
- new net MIDI_OUT: R12.1, U_CTRL.41
- new net MISO: ISP1.1, U_CTRL.11, U_SD.7
- new net MOSI: ISP1.4, U_CTRL.10, U_SD.3
- new net N$30: CD2.2, U_CTRL.17, Y1.P$2
- new net N$31: CD3.2, U_CTRL.16, Y1.P$1
- new net N$32: R20.1, U_CTRL.4
- new net N$33: R21.2, U_CTRL.33
- new net OUT1: C9.1, U1.1, VR1.3
- new net OUT2: C10.2, U1.7, VR1.5
- new net RST: BUTTON5.P$1, ISP1.5, U_CTRL.13
- new net SCK: ISP1.3, U_CTRL.9, U_SD.5
- new net SD_CS: U_CTRL.25, U_SD.2
- new net USB_D+: R20.2, U$43.A6, U$43.B6
- new net USB_D-: R19.2, U$43.A7, U$43.B7
- new net VBUS: C3.1, C6.1, D2.C, LED3.A, POWER_SW.1, U$43.A4B9, U$43.B4A9, U2.4, U3.1
- net +3V3: now also BUTTON1.P$1, BUTTON2.P$1, BUTTON3.P$1, BUTTON4.P$1, C14.1, C5.1, C7.1, ISP1.2, J4.1, J4.5, J4.8, R22.1, U1.8, U3.5, U_CTRL.14, U_CTRL.2, U_CTRL.24, U_CTRL.34, U_CTRL.44, U_CTRL.6, U_CTRL.7
- net CA11: now also C12.1; no longer CA12.1
- net ENABLE: now also POWER_SW.2, R9.2; no longer U1.11
- net GND: now also BUTTON5.P$2, C13.2, C14.2, CA2.2, CA6.2, CD2.1, CD3.1, ISP1.6, J1.1, J2.1, J3.2, J4.4, J4.MP1, J4.MP2, POWER_SW.3, R10.1, R15.1, R16.1, R21.1, R3.1, R7.1, U$1.P42, U$1.P43, U$1.P44, U1.4, U3.2, U_CTRL.15, U_CTRL.23, U_CTRL.35, U_CTRL.43, U_CTRL.5, U_SD.6, U_SD.MT1, U_SD.MT2, VR1.1, VR1.MH1, VR1.MH2, VR1.MP1, VR1.MP2; no longer B1.1, C8.-, LBO.C, R15.2, R18.1, R2.1, SD1.G0, SD1.G1, SD1.PIN6, U1.10, U1.13, U1.6, U1.7, U1.P$18, U1.P$19, U1.P$20, U1.P$21, U1.P$22, U1.THERMAL
- net LCD_A: now also R22.2
- net N$1: now also C9.2, J1.2; no longer JP1.2, R12.1
- net N$10: now also C11.2; no longer CA11.2
- net N$11: now also C12.2; no longer CA12.2
- net N$14: now also R2.1, U1.2
- net N$16: now also R18.1, U1.6
- net N$19: now also R9.1, U3.3; no longer L1.P$2, U1.3, U1.4
- net N$21: now also BUTTON1.P$2, R10.2, U_CTRL.12; no longer R18.2, R19.1, U1.9
- net N$22: now also BUTTON2.P$2, R15.2, U_CTRL.30; no longer PWR.C, R15.1
- net N$23: now also BUTTON3.P$2, R16.2, U_CTRL.29; no longer R16.1, R17.2, U1.14
- net N$24: now also BUTTON4.P$2, R17.2, U_CTRL.28; no longer U$10.P$2
- net N$25: now also C10.1, J1.3; no longer U$12.P$2
- net N$26: now also R2.2, VR1.2; no longer LBO.A, R20.1
- net N$27: now also C13.1, U1.3; no longer Q1.C, R20.2
- net N$28: now also R19.1, U_CTRL.3; no longer U$35.P$2
- net N$29: now also R18.2, VR1.4; no longer U$36.P$2
- net N$3: now also Y2.P$1; no longer Q2.2
- net N$5: now also Y2.P$2; no longer Q2.1
- net N$8: now also C11.1; no longer CA11.1
- net VBAT: now also D2.A, J2.2; no longer B1.2, C3.1, C7.1, L1.P$1, Q1.E, R19.2, U1.8
Routing:
- net VBUS: track 0.00 -> 108.3 mm, vias 0 -> 1
- net ENABLE: track 0.00 -> 81.1 mm, vias 0 -> 1
- net GND: track 0.00 -> 74.7 mm, vias 0 -> 14
- net N$21: track 0.00 -> 73.1 mm, vias 0 -> 5
- net +3V3: track 0.00 -> 66.7 mm, vias 0 -> 19
- net N$22: track 0.00 -> 45.3 mm, vias 0 -> 1
- net N$6: track 0.00 -> 41.7 mm, vias 0 -> 2
- net N$28: track 0.00 -> 40.2 mm, vias 0 -> 2
- net N$32: track 0.00 -> 39.4 mm, vias 0 -> 2
- net OUT2: track 0.00 -> 35.8 mm, vias 0 -> 2
- net OUT1: track 0.00 -> 34.6 mm, vias 0 -> 2
- net N$23: track 0.00 -> 34.1 mm, vias 0 -> 1
- net MISO: track 0.00 -> 32.3 mm
- net N$16: track 0.00 -> 31.2 mm, vias 0 -> 2
- net SD_CS: track 0.00 -> 29.0 mm, vias 0 -> 2
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- added copper zone on layer 1, net +3V3
- added copper zone on layer 16, net GND
- added copper zone on layer 1, net N$34
Other:
- board size 45 x 85 mm -> 45.2 x 69.2 mm
- board text added: "RESET"
- board text added: "https://www.adafruit.com/product/1317"

Commit message: made the midipod I can build
Parts:
- removed D2: MBR120, diode:SMB
- removed U_SD: MICROSD, adafruit:MICROSD
- removed Y1: 16MHz, SparkFun-Clocks:CRYSTAL-SMD-3.2X1.5MM
- added D3: MBR120, adafruit:SOD-123
- added J5: 104031-0811, SamacSys_Parts:1040310811
- added Y3: 407F35E009M6000, SamacSys_Parts:407F35E009M6000
- Y2: value 9.6MHz -> ABM8-16.000MHZ-D1X-T; device SparkFun-Clocks:CRYSTAL-SMD-3.2X1.5MM -> SamacSys_Parts:ABM816000MHZD1XT
- moved Y2 30.2 mm to (38.6, 51.7), turned to 0 degrees
- moved ISP1 7.50 mm to (24.4, 62.6)
- moved C2 7.26 mm to (5.41, 30.8)
- moved C1 7.08 mm to (5.41, 32.7)
- moved CD3 3.26 mm to (37.0, 54.6), turned to 0 degrees
- moved CD2 3.12 mm to (40.3, 54.6)
- moved CD5 2.00 mm to (3.93, 35.8)
- moved CD6 2.00 mm to (3.96, 37.8)
- moved BUTTON5 1.97 mm to (18.6, 61.5)
Connections:
- removed net N$30: CD2.2, U_CTRL.17, Y1.P$2
- removed net N$31: CD3.2, U_CTRL.16, Y1.P$1
- new net N$35: CD2.2, U_CTRL.17, Y2.1
- new net N$36: CD3.2, U_CTRL.16, Y2.3
- net +3V3: now also J5.4
- net 7: no longer U_SD.CD1
- net GND: now also J5.6, Y2.2, Y2.4, Y3.2, Y3.4; no longer U_SD.6, U_SD.MT1, U_SD.MT2
- net MISO: now also J5.7; no longer U_SD.7
- net MOSI: now also J5.3; no longer U_SD.3
- net N$3: now also Y3.1; no longer Y2.P$1
- net N$5: now also Y3.3; no longer Y2.P$2
- net SCK: now also J5.5; no longer U_SD.5
- net SD_CS: now also J5.2; no longer U_SD.2
- net VBAT: now also D3.A; no longer D2.A
- net VBUS: now also D3.C; no longer D2.C
Routing:
- net 7: track 20.4 -> 0.00 mm, vias 2 -> 0
- net SCK: track 23.4 -> 34.9 mm, vias 0 -> 1
- net N$35: track 0.00 -> 9.95 mm
- net GND: track 74.7 -> 64.8 mm, vias 14 -> 13
- net N$36: track 0.00 -> 9.37 mm
- net +3V3: track 66.7 -> 75.5 mm, vias 19 -> 20
- net N$3: track 5.40 -> 13.6 mm
- net N$30: track 7.16 -> 0.00 mm
- net MOSI: track 20.1 -> 26.8 mm
- net N$5: track 4.83 -> 11.3 mm
- net N$31: track 5.82 -> 0.00 mm
- net MISO: track 32.3 -> 37.0 mm, vias 0 -> 2
- net SD_CS: track 29.0 -> 24.8 mm
- net N$6: track 41.7 -> 43.7 mm
- net VBAT: track 22.0 -> 20.4 mm
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