File: MIDIpod.sch (EAGLE design)
At the start: 59 parts, among them IC1 TPA6132A2, J1 SJ-3524-SMT-TR, J4 68610814122, Q1 MMUN2133LT1G, Q2 9.6MHz, U1 TPS61090RSAR, U2 MCP73831T-2ACI/OT

Commit message: updated, sent to oshpark
Parts:
- removed B1: 1.8-5V, microbuilder:BATTERY
- removed IC1: TPA6132A2, texas:TPA6132A2
- removed JP1: (no value), pinhead:PINHD-1X3
- removed L1: VLC5045-6.8uH, microbuilder:INDUCTORTDK_VLC5045
- removed LBO: RED, microbuilder:LED0805_NOOUTLINE
- removed PWR: BLUE, microbuilder:LED0805_NOOUTLINE
- removed Q1: MMUN2133LT1G, transistor:MUN2114T1-PNP_DRIVER-SC59-BEC
- removed Q2: 9.6MHz, crystal:CRYSTALTC26H
- removed SD1: MF-MICROSD, MF_Connectors:SD_CARD_SLOT_MICRO_RIGHT
- removed U$10, U$12, U$35, U$36: 1U_PAD, SiliconeSwitches:1U_PAD
- removed U$13: ATMEGA32U4-AU, adafruit:ATMEGA32U4-AU
- added BUTTON1, BUTTON2, BUTTON3, BUTTON4, BUTTON5: 1U_PAD, SiliconeSwitches:1U_PAD
- added C10, C9: 2.2pF, rcl:C-EUC0603
- added C13, C14: 1uF, SparkFun-Capacitors:0.1UF-0402-16V-10%
- added CD2, CD3: 22pf, rcl:C-EUC0603
- added D2: MBR120, diode:MBRS130LT3
- added ISP1: AVRISP-6, adafruit:AVRISP-6
- added J2: (no value), SparkFun-Connectors:CONN_02
- added POWER_SW: ALPSSLIDESW, TindieBadge:ALPSSLIDESW
- added R10: 10k, rcl:R-EU_R0603
- added R21: 1k, rcl:R-EU_R0603
- added R22: 220, rcl:R-EU_R0603
- added R9: 100k, microbuilder:RESISTOR0805_NOOUTLINE
- added U3: SPX3819M5_3_3, SparkFun-IC-Power:V_REG_SPX3819-SOT23-5
- added U_CTRL: ATMEGA32U4-AU, adafruit:ATMEGA32U4-AU
- added U_SD: MICROSD, adafruit:MICROSD
- added Y1: 16MHz, SparkFun-Clocks:CRYSTALSMD-3.2X1.5
- added Y2: 9.6MHz, SparkFun-Clocks:CRYSTALSMD-3.2X1.5
- C3: value 10uF -> 10µF
- C5: value 2.2uF -> 10µF
- C7: value 0.1uF -> 1uF
- C8: value 100uF/6V -> 2.2uF; device microbuilder:CAP_TANTALUMB/3528_REFLOW -> SparkFun-Capacitors:2.2UF-0805-25V-(+80/-20%)
- R15: value 1K -> 10k; device microbuilder:RESISTOR0805_NOOUTLINE -> rcl:R-EU_R0603
- R16: value 1.87Mohm -> 10k; device microbuilder:RESISTOR0805_NOOUTLINE -> rcl:R-EU_R0603
- R17: value 200K -> 10k; device microbuilder:RESISTOR0805_NOOUTLINE -> rcl:R-EU_R0603
- R18: value 340K -> 220; device microbuilder:RESISTOR0805_NOOUTLINE -> rcl:R-EU_R0603
- R19: value 1.87Mohm -> 22; device microbuilder:RESISTOR0805_NOOUTLINE -> rcl:R-EU_R0603
- R2: value 0 -> 220
- R20: value 1K -> 22; device microbuilder:RESISTOR0805_NOOUTLINE -> rcl:R-EU_R0603
- U1: value TPS61090RSAR -> TPA6111A2DR; device microbuilder:VREG_TPS6103X -> SparkFun-IC-Amplifiers:TPA6111SMD-T
- renumbered CA11 to C11, CA12 to C12
Connections:
- removed net 5.0V: C5.1, C8.+, PWR.A, R16.2, U1.VOUT
- removed net AGND: CA2.2, CA6.2, R2.2, R3.1, R7.1, U$1.AGND, U$1.AGND2, U$1.AGNDREF
- removed net LBO: Q1.B, U1.LBO
- removed net LCD_K: J3.2
- removed net PIN4: JP1.1
- removed net TXD: JP1.3
- removed net VDD1: C6.1, LED3.A, U$43.VBUS, U2.VDD
- new net 7: U_CTRL.PE6(INT.6/AIN0), U_SD.CARD_DETECT
- new net LCD_CAP1N: C8.2, J4.7
- new net LCD_CAP1P: C8.1, J4.6
- new net LCD_SCL: J4.2, U_CTRL.PD0(INT0/OC0B/SCL)
- new net LCD_SDA: J4.3, U_CTRL.PD1(INT1/SDA)
- new net MIDI_OUT: R12.1, U_CTRL.PF0(ADC0)
- new net MISO: ISP1.MISO, U_CTRL.PB3(PDO/MISO), U_SD.DATA_OUT
- new net MOSI: ISP1.MOSI, U_CTRL.PB2(PDI/MOSI), U_SD.DATA_IN
- new net N$30: CD2.2, U_CTRL.XTAL1, Y1.2
- new net N$31: CD3.2, U_CTRL.XTAL2, Y1.1
- new net N$32: R20.1, U_CTRL.D+
- new net N$33: R21.2, U_CTRL.PE2(!HWB)
- new net OUT1: C9.1, U1.VO1, VR1.3_1
- new net OUT2: C10.2, U1.VO2, VR1.3_2
- new net RST: BUTTON5.P$1, ISP1.RST, U_CTRL./RESET
- new net SCK: ISP1.SCK, U_CTRL.PB1(SCK), U_SD.SCLK
- new net SD_CS: U_CTRL.PD4(ICP1/ADC8), U_SD.CS
- new net USB_D+: R20.2, U$43.DP1, U$43.DP2
- new net USB_D-: R19.2, U$43.DN1, U$43.DN2
- new net VBUS: C3.1, C6.1, D2.C, LED3.A, POWER_SW.1, U$43.VBUS, U2.VDD, U3.IN
- net +3V3: now also BUTTON1.P$1, BUTTON2.P$1, BUTTON3.P$1, BUTTON4.P$1, C14.1, C5.1, C7.1, ISP1.VCC, J4.1, J4.5, J4.8, R22.1, U1.VDD, U3.OUT, U_CTRL.AVCC, U_CTRL.AVCC1, U_CTRL.UCAP, U_CTRL.UVCC, U_CTRL.VBUS, U_CTRL.VCC, U_CTRL.VCC1
- net ENABLE: now also POWER_SW.2, R9.2; no longer U1.EN
- net GND: now also BUTTON5.P$2, C13.2, C14.2, CA2.2, CA6.2, CD2.1, CD3.1, ISP1.GND, J1.SLEEVE, J2.1, J3.2, J4.4, J4.MP1, J4.MP2, POWER_SW.3, R10.1, R15.1, R16.1, R21.1, R3.1, R7.1, U$1.AGND, U$1.AGND2, U$1.AGNDREF, U1.SHT, U3.GND, U_CTRL.GND, U_CTRL.GND1, U_CTRL.GND2, U_CTRL.GND3, U_CTRL.UGND, U_SD.GND, U_SD.GND1, U_SD.VSS, VR1.1/1, VR1.MH1, VR1.MH2, VR1.MP1, VR1.MP2; no longer B1.-, C8.-, LBO.C, R15.2, R18.1, R2.1, U1.PGND, U1.SYNC
- net LCD_A: now also R22.2
- net N$1: now also C9.2, J1.TIP; no longer JP1.2, R12.1
- net N$14: now also R2.1, U1.IN1
- net N$16: now also R18.1, U1.IN2
- net N$19: now also R9.1, U3.EN; no longer L1.2, U1.SW
- net N$21: now also BUTTON1.P$2, R10.2, U_CTRL.PB7(OC0A/OC1C/RTS); no longer R18.2, R19.1, U1.LBI
- net N$22: now also BUTTON2.P$2, R15.2, U_CTRL.PB6(OC1B/OC4B/ADC13); no longer PWR.C, R15.1
- net N$23: now also BUTTON3.P$2, R16.2, U_CTRL.PB5(OC1A/ADC12/!OC4B); no longer R16.1, R17.2, U1.FB
- net N$24: now also BUTTON4.P$2, R17.2, U_CTRL.PB4(ADC11); no longer U$10.P$2
- net N$25: now also C10.1, J1.RING; no longer U$12.P$2
- net N$26: now also R2.2, VR1.2_1; no longer LBO.A, R20.1
- net N$27: now also C13.1, U1.BYP; no longer Q1.C, R20.2
- net N$28: now also R19.1, U_CTRL.D-; no longer U$35.P$2
- net N$29: now also R18.2, VR1.2_2; no longer U$36.P$2
- net N$3: now also Y2.1; no longer Q2.2
- net N$5: now also Y2.2; no longer Q2.1
- net VBAT: now also D2.A, J2.2; no longer B1.+, C3.1, C7.1, L1.1, Q1.E, R19.2, U1.VBAT
Other:
- note removed: "6.8uH power w/2A current"
- note removed: "R2 < 500K R1 = 5.5*R2 (3.2V LBO)"
- note removed: "R4 = 200K R3 = 1.85Mohm"
- note removed: "See Pg 15 1st para"
- moved on the sheet: C3, C5, C6, C7, J1, J3, J4, LED3, LED4, R11, R13, R14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

Commit message: made the midipod I can build
Parts:
- removed D2: MBR120, diode:MBRS130LT3
- removed U_SD: MICROSD, adafruit:MICROSD
- removed Y1: 16MHz, SparkFun-Clocks:CRYSTALSMD-3.2X1.5
- added D3: MBR120, adafruit:DIODESOD-123
- added J5: 104031-0811, SamacSys_Parts:104031-0811
- added Y3: 407F35E009M6000, SamacSys_Parts:407F35E009M6000
- Y2: value 9.6MHz -> ABM8-16.000MHZ-D1X-T; device SparkFun-Clocks:CRYSTALSMD-3.2X1.5 -> SamacSys_Parts:ABM8-16.000MHZ-D1X-T
Connections:
- removed net N$30: CD2.2, U_CTRL.XTAL1, Y1.2
- removed net N$31: CD3.2, U_CTRL.XTAL2, Y1.1
- new net N$35: CD2.2, U_CTRL.XTAL1, Y2.CRYSTAL_1
- new net N$36: CD3.2, U_CTRL.XTAL2, Y2.CRYSTAL_2
- net +3V3: now also J5.VDD
- net 7: no longer U_SD.CARD_DETECT
- net GND: now also J5.VSS, Y2.GND_1, Y2.GND_2, Y3.GND_1, Y3.GND_2; no longer U_SD.GND, U_SD.GND1, U_SD.VSS
- net MISO: now also J5.DAT0; no longer U_SD.DATA_OUT
- net MOSI: now also J5.CMD; no longer U_SD.DATA_IN
- net N$3: now also Y3.CRYSTAL_1; no longer Y2.1
- net N$5: now also Y3.CRYSTAL_2; no longer Y2.2
- net SCK: now also J5.CLK; no longer U_SD.SCLK
- net SD_CS: now also J5.CD/DAT3; no longer U_SD.CS
- net VBAT: now also D3.A; no longer D2.A
- net VBUS: now also D3.C; no longer D2.C
Other:
- moved on the sheet: C2
